File: Hardware/Brushless_ESC_STC_V2/Brushless_ESC_STC_V2.kicad_pcb (KiCad board)
At the start: 4 copper layers, 37.6 x 25.4 mm, 57 parts, among them J1 Conn_01x01_Male, J2 Conn_01x01_Male, J3 Conn_01x01_Male, J4 Conn_01x04_Male, J5 Conn_01x01_Male, J6 Conn_01x01_Male, J7 Conn_01x01_Male, J8 Conn_01x01_Male, J9 Conn_01x01_Male, Q1 S8050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

Commit message: ESCV2生成制板文件
Other:
- board text added: "ESC By Del"
